Commit message: Draw the links with meshes, and ship them as package:// paths
Generate one mesh per section from the robot config: the real link shape,
with a flat top and a bottom cut by the rolling arc of radius R, plus a
second mesh per section that marks the rod holes as dark discs.

rollchain_urdf generates the meshes and expands the xacro with them, so the
URDF, the meshes and the model always come from the same config. The build
generates a set for every config in rollchain_description/config and installs
it under share/rollchain_description/meshes/<geometry hash>; the URDF then
references them as package:// paths, which resolve on any machine with the
package installed, so robot_description can go to an RViz elsewhere. A config
from outside the package has nothing installed to point at, so it falls back
to a local cache with file:// paths and a note on stderr.

Rods gain an optional w, the depth along the joint axis: it keeps the holes
apart and places them in the drawing, but does not enter the planar statics.
Validation now also rejects two holes that overlap.

Co-Authored-By: Claude Opus 5 <noreply@anthropic.com>

File: src/rollchain_description/urdf/rollchain.urdf.xacro (robot description, xacro)
@@ -14,11 +14,19 @@
   The real joint range is computed and enforced by the model (theory RC5);
   the URDF limits are deliberately generous so there is no second copy of it.
+  Visuals: with mesh_uri set to a URI prefix (rollchain_urdf does this, with
+  the package:// path of the installed meshes, or a local cache URI for a config
+  the package does not ship), each link is drawn with <mesh_uri>/section_{s}.stl,
+  its real shape with the rolling arc, plus section_{s}_holes.stl for the rod
+  holes. Without it, plain cylinders.
 -->
 <robot name="rollchain" xmlns:xacro="http://www.ros.org/wiki/xacro">
   <xacro:arg name="config" default="$(find rollchain_description)/config/reference_robot.yaml"/>
+  <xacro:arg name="mesh_uri" default=""/>
   <xacro:property name="cfg" value="${xacro.load_yaml('$(arg config)')['/**']['ros__parameters']}"/>
   <xacro:property name="sec" value="${cfg['sections']}"/>
   <xacro:property name="num_sections" value="${len(sec['n'])}"/>
   <xacro:property name="base_length" value="${cfg['base']['length']}"/>
+  <xacro:property name="mesh_uri" value="$(arg mesh_uri)"/>
+  <xacro:property name="use_meshes" value="${len(mesh_uri) > 0}"/>
   <material name="rc_base"><color rgba="0.40 0.40 0.40 1"/></material>
   <material name="rc_0"><color rgba="0.85 0.45 0.15 1"/></material>
@@ -27,4 +35,5 @@
   <material name="rc_3"><color rgba="0.60 0.35 0.70 1"/></material>
   <material name="rc_4"><color rgba="0.80 0.30 0.30 1"/></material>
+  <material name="rc_hole"><color rgba="0.08 0.08 0.08 1"/></material>
   <link name="base_link">
     <visual>
@@ -68,14 +77,30 @@
       <origin xyz="0 0 ${-R}"/>
     </joint>
-    <!-- Visual: a cylinder from the crest to the flat top, coloured by section.
-         Replace it with a mesh of the real link (flat top, one bottom arc) when you have one. -->
+    <!-- Visual, coloured by section: the real link shape (mesh in the link frame,
+         origin at the crest), or a cylinder from the crest to the flat top. -->
     <link name="link_${i}">
-      <visual>
-        <origin xyz="0 0 ${L / 2}"/>
-        <geometry>
-          <cylinder radius="${D / 2}" length="${L}"/>
-        </geometry>
-        <material name="rc_${s % 5}"/>
-      </visual>
+      <xacro:if value="${use_meshes}">
+        <visual>
+          <geometry>
+            <mesh filename="${mesh_uri}/section_${s + 1}.stl"/>
+          </geometry>
+          <material name="rc_${s % 5}"/>
+        </visual>
+        <visual>
+          <geometry>
+            <mesh filename="${mesh_uri}/section_${s + 1}_holes.stl"/>
+          </geometry>
+          <material name="rc_hole"/>
+        </visual>
+      </xacro:if>
+      <xacro:unless value="${use_meshes}">
+        <visual>
+          <origin xyz="0 0 ${L / 2}"/>
+          <geometry>
+            <cylinder radius="${D / 2}" length="${L}"/>
+          </geometry>
+          <material name="rc_${s % 5}"/>
+        </visual>
+      </xacro:unless>
     </link>
     <xacro:if value="${k &lt; n}">
